Commit message: Giant leap

File: description/robot.urdf.xacro (robot description, xacro)
@@ -2,3 +2,5 @@
 <robot xmlns:xacro="http://www.ros.org/wiki/xacro"  name="robot">
     <xacro:include filename="robot_core.xacro" />
+    <!-- <xacro:include filename="ros2_control.xacro" /> -->
+    <xacro:include filename="gazebo_control.xacro" />
 </robot>

File: description/robot_core.xacro (robot description, xacro)
@@ -28,7 +28,7 @@
             <origin rpy="${pi/2} 0 ${pi/2}" xyz="0 0 0"/>
             <geometry>
-                <mesh filename="package://meshes/chassis.stl" scale="0.001 0.001 0.001"/>
+                <mesh filename="package://robot_one/meshes/chassis.stl" scale="0.001 0.001 0.001"/>
             </geometry>
-            <material name="white"/>
+            <material name="Gazebo/white"/>
         </visual>
         <!-- <collision>
@@ -52,7 +52,7 @@
             <origin xyz="0 0 0" rpy="${pi/2} 0 ${pi}"/>
             <geometry>
-                <mesh filename="package://meshes/gearbox.stl" scale="0.001 0.001 0.001"/>
+                <mesh filename="package://robot_one/meshes/gearbox.stl" scale="0.001 0.001 0.001"/>
             </geometry>
-            <material name="blue"/>
+            <material name="Gazebo/blue"/>
         </visual>
         <!-- <collision>
@@ -74,7 +74,7 @@
         <visual>
             <geometry>
-                <mesh filename="package://meshes/gearbox.stl" scale="0.001 0.001 0.001"/>
+                <mesh filename="package://robot_one/meshes/gearbox.stl" scale="0.001 0.001 0.001"/>
             </geometry>
-            <material name="blue"/>
+            <material name="Gazebo/blue"/>
         </visual>
         <!-- <collision>
@@ -113,3 +113,9 @@
     <xacro:caster_wheel_joint prefix="rear_right" origin="-0.22 -0.178 -0.005"/>
     <xacro:caster_wheel prefix="rear_right"/>
+    <gazebo>
+    <plugin filename="libgazebo_gazebo_system.so" name="gazebo_ros2_control">
+        <robot_sim_type>gazebo_ros2_control/GazeboSystem</robot_sim_type>
+        <parameters>/home/sss0301/ros2_ws/src/robot_one/config/robot_control.yaml</parameters>
+    </plugin>
+    </gazebo>
 </robot>

Commit message: start ros2_control

File: description/robot.urdf.xacro (robot description, xacro)
@@ -2,5 +2,5 @@
 <robot xmlns:xacro="http://www.ros.org/wiki/xacro"  name="robot">
     <xacro:include filename="robot_core.xacro" />
-    <!-- <xacro:include filename="ros2_control.xacro" /> -->
-    <xacro:include filename="gazebo_control.xacro" />
+    <xacro:include filename="ros2_control.xacro" />
+    <!-- <xacro:include filename="gazebo_control.xacro" /> -->
 </robot>

File: description/robot_core.xacro (robot description, xacro)
@@ -87,5 +87,5 @@
     </link>
     <joint name="right_wheel_joint" type="continuous">
-        <origin xyz="0 0.1715 0.01" rpy="${pi/2} 0 0"/>
+        <origin xyz="0 0.1715 0.015" rpy="${pi/2} 0 0"/>
         <axis xyz="0 0 1" rpy="0 0 0"/>
         <parent link="base_link"/>
@@ -96,5 +96,5 @@
     <xacro:wheel_link prefix="right"/>
     <joint name="left_wheel_joint" type="continuous">
-        <origin xyz="0 -0.1715 0.01" rpy="${pi/2} 0 0"/>
+        <origin xyz="0 -0.1715 0.015" rpy="${pi/2} 0 0"/>
         <axis xyz="0 0 1" rpy="0 0 0"/>
         <parent link="base_link"/>
@@ -112,9 +112,3 @@
     <xacro:caster_wheel_joint prefix="rear_right" origin="-0.22 -0.178 -0.005"/>
     <xacro:caster_wheel prefix="rear_right"/>
-    <gazebo>
-    <plugin filename="libgazebo_gazebo_system.so" name="gazebo_ros2_control">
-        <robot_sim_type>gazebo_ros2_control/GazeboSystem</robot_sim_type>
-        <parameters>/home/sss0301/ros2_ws/src/robot_one/config/robot_control.yaml</parameters>
-    </plugin>
-    </gazebo>
 </robot>

File: description/ros2_control.xacro (robot description, xacro)
@@ -2,23 +2,28 @@
 <robot xmlns:xacro="http://www.ros.org/wiki/xacro"  name="ros2_control">
     <ros2_control name="GazeboSystem" type="system">
-    <hardware>
-        <plugin>gazebo_ros2_control/GazeboSystem</plugin>
-    </hardware>
-    <joint name="left_wheel_joint">
-        <command_interface name="velocity">
-            <param name="min">-10</param>
-            <param name="max">10</param>
-        </command_interface>
-        <state_interface name="position" />
-        <state_interface name="velocity" />
-    </joint>
-    <joint name="right_wheel_joint">
-        <command_interface name="velocity">
-            <param name="min">-10</param>
-            <param name="max">10</param>
-        </command_interface>
-        <state_interface name="velocity" />
-        <state_interface name="position" />
-    </joint>
-</ros2_control>
+        <hardware>
+            <plugin>gazebo_ros2_control/GazeboSystem</plugin>
+        </hardware>
+        <joint name="left_wheel_joint">
+            <command_interface name="velocity">
+                <param name="min">-10</param>
+                <param name="max">10</param>
+            </command_interface>
+            <state_interface name="position" />
+            <state_interface name="velocity" />
+        </joint>
+        <joint name="right_wheel_joint">
+            <command_interface name="velocity">
+                <param name="min">-10</param>
+                <param name="max">10</param>
+            </command_interface>
+            <state_interface name="velocity" />
+            <state_interface name="position" />
+        </joint>
+    </ros2_control>
+    <gazebo>
+        <plugin filename="libgazebo_gazebo_system.so" name="gazebo_ros2_control">
+            <parameters>$(find robot_one)/config/robot_control.yaml</parameters>
+        </plugin>
+    </gazebo>
 </robot>
