Commit message: robot base done(only origin)

File: description/robot_core.xacro (robot description, xacro)
@@ -65,6 +65,4 @@
         </xacro:inertial_cylinder>
     </link>
-    <xacro:wheel_joint prefix="left" origin="0 0.045 0.04"/>
-    <xacro:wheel prefix="left"/>
     <!-- RIGHT WHEEL LINK -->
     <joint name="right_gearbox_joint" type="fixed">
@@ -89,5 +87,29 @@
         </xacro:inertial_cylinder> -->
     </link>
-    <xacro:wheel_joint prefix="right" origin="0 -0.045 0.04"/>
-    <xacro:wheel prefix="right"/>
+    <joint name="right_wheel_joint" type="continuous">
+        <origin xyz="0 -0.1715 0" rpy="${pi/2} 0 0"/>
+        <axis xyz="0 0 1"/>
+        <parent link="base_link"/>
+        <child link="right_wheel"/>
+        <!-- right xyz="0 -0.045 0.04" -->
+        <!-- left xyz="0 0.045 0.04" -->
+    </joint>
+    <xacro:wheel_link prefix="right"/>
+    <joint name="left_wheel_joint" type="continuous">
+        <origin xyz="0 0.1715 0" rpy="${pi/2} 0 0"/>
+        <axis xyz="0 0 1"/>
+        <parent link="base_link"/>
+        <child link="left_wheel"/>
+        <!-- right xyz="0 -0.045 0.04" -->
+        <!-- left xyz="0 0.045 0.04" -->
+    </joint>
+    <xacro:wheel_link prefix="left"/>
+    <xacro:caster_wheel_joint prefix="front_left" origin="0.22 0.178 -0.005"/>
+    <xacro:caster_wheel prefix="front_left"/>
+    <xacro:caster_wheel_joint prefix="front_right" origin="0.22 -0.178 -0.005"/>
+    <xacro:caster_wheel prefix="front_right"/>
+    <xacro:caster_wheel_joint prefix="rear_left" origin="-0.22 0.178 -0.005"/>
+    <xacro:caster_wheel prefix="rear_left"/>
+    <xacro:caster_wheel_joint prefix="rear_right" origin="-0.22 -0.178 -0.005"/>
+    <xacro:caster_wheel prefix="rear_right"/>
 </robot>

File: description/robot_essential.xacro (robot description, xacro)
@@ -1,17 +1,6 @@
 <?xml version="1.0"?>
 <robot xmlns:xacro="http://www.ros.org/wiki/xacro" name="robot_essential">
-    <!-- WHEEL JOINT -->
-    <xacro:macro name="wheel_joint" params="prefix origin">
-        <joint name="${prefix}_wheel_joint" type="fixed">
-            <origin xyz="${origin}" rpy="0 0 0"/>
-            <axis xyz="0 1 0"/>
-            <parent link="${prefix}_gearbox"/>
-            <child link="${prefix}_wheel"/>
-            <!-- right xyz="0 -0.045 0.04" -->
-            <!-- left xyz="0 0.045 0.04" -->
-        </joint>
-    </xacro:macro>
     <!-- WHEEL LINK -->
-    <xacro:macro name="wheel" params="prefix">
+    <xacro:macro name="wheel_link" params="prefix">
         <link name="${prefix}_wheel">
             <visual>
@@ -49,11 +38,11 @@
         </link>
     </xacro:macro>
-    <!-- CASTER WHEEL LINK -->
-    <!-- <xacro:macro name="caster_wheel_joint">
-        <joint name="caster_wheel_joint" type="fixed">
-            <parent link="chassis"/>
-            <child link="caster_wheel"/>
-            <origin xyz="0.24 0 0"/>
+    <!-- Caster Wheel JOINT -->
+    <xacro:macro name="caster_wheel_joint" params="prefix origin">
+        <joint name="${prefix}_caster_wheel_joint" type="fixed">
+            <parent link="base_link"/>
+            <child link="${prefix}_caster_wheel"/>
+            <origin xyz="${origin}"/>
         </joint>
-    </xacro:macro> -->
+    </xacro:macro>
 </robot>

Commit message: gazebo plugin

File: description/robot_core.xacro (robot description, xacro)
@@ -89,5 +89,5 @@
     <joint name="right_wheel_joint" type="continuous">
         <origin xyz="0 -0.1715 0" rpy="${pi/2} 0 0"/>
-        <axis xyz="0 0 1"/>
+        <axis xyz="0 0 1" rpy="0 0 0"/>
         <parent link="base_link"/>
         <child link="right_wheel"/>
@@ -98,5 +98,5 @@
     <joint name="left_wheel_joint" type="continuous">
         <origin xyz="0 0.1715 0" rpy="${pi/2} 0 0"/>
-        <axis xyz="0 0 1"/>
+        <axis xyz="0 0 1" rpy="0 0 0"/>
         <parent link="base_link"/>
         <child link="left_wheel"/>
@@ -113,3 +113,9 @@
     <xacro:caster_wheel_joint prefix="rear_right" origin="-0.22 -0.178 -0.005"/>
     <xacro:caster_wheel prefix="rear_right"/>
+    <gazebo>
+    <plugin filename="libgazebo_ros2_control.so" name="gazebo_ros2_control">
+        <robot_sim_type>gazebo_ros2_control/GazeboSystem</robot_sim_type>
+        <parameters>/home/lin/gazebo_ros2_control/src/r2d/config/r2d_joint_trajectory.yaml</parameters>
+    </plugin>
+    </gazebo>
 </robot>

Commit message: nOO

File: description/robot_core.xacro (robot description, xacro)
@@ -28,5 +28,5 @@
             <origin rpy="${pi/2} 0 ${pi/2}" xyz="0 0 0"/>
             <geometry>
-                <mesh filename="package://robot_one/meshes/chassis.stl" scale="0.001 0.001 0.001"/>
+                <mesh filename="$(find robot_one)/meshes/chassis.stl" scale="0.001 0.001 0.001"/>
             </geometry>
             <material name="white"/>
@@ -52,5 +52,5 @@
             <origin xyz="0 0 0" rpy="${pi/2} 0 ${pi}"/>
             <geometry>
-                <mesh filename="package://robot_one/meshes/gearbox.stl" scale="0.001 0.001 0.001"/>
+                <mesh filename="$(find robot_one)/meshes/gearbox.stl" scale="0.001 0.001 0.001"/>
             </geometry>
             <material name="blue"/>
@@ -74,5 +74,5 @@
         <visual>
             <geometry>
-                <mesh filename="package://robot_one/meshes/gearbox.stl" scale="0.001 0.001 0.001"/>
+                <mesh filename="$(find robot_one)/meshes/gearbox.stl" scale="0.001 0.001 0.001"/>
             </geometry>
             <material name="blue"/>
@@ -113,9 +113,3 @@
     <xacro:caster_wheel_joint prefix="rear_right" origin="-0.22 -0.178 -0.005"/>
     <xacro:caster_wheel prefix="rear_right"/>
-    <gazebo>
-    <plugin filename="libgazebo_ros2_control.so" name="gazebo_ros2_control">
-        <robot_sim_type>gazebo_ros2_control/GazeboSystem</robot_sim_type>
-        <parameters>/home/sss0301/ros2_ws/src/robot_one/config/robot_control.yaml</parameters>
-    </plugin>
-    </gazebo>
 </robot>

Commit message: add gazebo launch file

File: description/robot_core.xacro (robot description, xacro)
@@ -28,5 +28,5 @@
             <origin rpy="${pi/2} 0 ${pi/2}" xyz="0 0 0"/>
             <geometry>
-                <mesh filename="$(find robot_one)/meshes/chassis.stl" scale="0.001 0.001 0.001"/>
+                <mesh filename="package://meshes/chassis.stl" scale="0.001 0.001 0.001"/>
             </geometry>
             <material name="white"/>
@@ -52,5 +52,5 @@
             <origin xyz="0 0 0" rpy="${pi/2} 0 ${pi}"/>
             <geometry>
-                <mesh filename="$(find robot_one)/meshes/gearbox.stl" scale="0.001 0.001 0.001"/>
+                <mesh filename="package://meshes/gearbox.stl" scale="0.001 0.001 0.001"/>
             </geometry>
             <material name="blue"/>
@@ -74,5 +74,5 @@
         <visual>
             <geometry>
-                <mesh filename="$(find robot_one)/meshes/gearbox.stl" scale="0.001 0.001 0.001"/>
+                <mesh filename="package://meshes/gearbox.stl" scale="0.001 0.001 0.001"/>
             </geometry>
             <material name="blue"/>

Commit message: Lower the wheel

File: description/robot_core.xacro (robot description, xacro)
@@ -33,10 +33,9 @@
         </visual>
         <!-- <collision>
-            <origin xyz="0.15 0 0.075"/>
             <geometry>
-                <box size="0.3 0.3 0.15"/>
+                <mesh filename="package://robot_one/meshes/gearbox.stl" scale="0.001 0.001 0.001"/>
             </geometry>
-        </collision>
-        <xacro:inertial_box mass="0.5" x="0.3" y="0.3" z="0.15">
+        </collision> -->
+        <!-- <xacro:inertial_box mass="0.5" x="0.3" y="0.3" z="0.15">
             <origin xyz="0.15 0 0.075" rpy="0 0 0"/>
         </xacro:inertial_box> -->
@@ -58,10 +57,10 @@
         <!-- <collision>
             <geometry>
-                <cylinder radius="0.05" length="0.04"/>
+               <mesh filename="package://robot_one/meshes/gearbox.stl" scale="0.001 0.001 0.001"/>
             </geometry>
         </collision> -->
-        <xacro:inertial_cylinder mass="0.1" length="0.04" radius="0.05">
+        <!-- <xacro:inertial_cylinder mass="0.1" length="0.04" radius="0.05">
             <origin xyz="0 0 0" rpy="0 0 0"/>
-        </xacro:inertial_cylinder>
+        </xacro:inertial_cylinder> -->
     </link>
     <!-- RIGHT WHEEL LINK -->
@@ -80,5 +79,5 @@
         <!-- <collision>
             <geometry>
-                <cylinder radius="0.05" length="0.04"/>
+                <mesh filename="package://robot_one/meshes/gearbox.stl" scale="0.001 0.001 0.001"/>
             </geometry>
         </collision> -->
@@ -88,5 +87,5 @@
     </link>
     <joint name="right_wheel_joint" type="continuous">
-        <origin xyz="0 -0.1715 0" rpy="${pi/2} 0 0"/>
+        <origin xyz="0 0.1715 0.01" rpy="${pi/2} 0 0"/>
         <axis xyz="0 0 1" rpy="0 0 0"/>
         <parent link="base_link"/>
@@ -97,5 +96,5 @@
     <xacro:wheel_link prefix="right"/>
     <joint name="left_wheel_joint" type="continuous">
-        <origin xyz="0 0.1715 0" rpy="${pi/2} 0 0"/>
+        <origin xyz="0 -0.1715 0.01" rpy="${pi/2} 0 0"/>
         <axis xyz="0 0 1" rpy="0 0 0"/>
         <parent link="base_link"/>

Commit message: move /meshes to /description

File: description/robot_core.xacro (robot description, xacro)
@@ -28,5 +28,5 @@
             <origin rpy="${pi/2} 0 ${pi/2}" xyz="0 0 0"/>
             <geometry>
-                <mesh filename="package://robot_one/meshes/chassis.stl" scale="0.001 0.001 0.001"/>
+                <mesh filename="package://robot_one/description/meshes/chassis.stl" scale="0.001 0.001 0.001"/>
             </geometry>
             <material name="Gazebo/white"/>
@@ -34,5 +34,5 @@
         <!-- <collision>
             <geometry>
-                <mesh filename="package://robot_one/meshes/gearbox.stl" scale="0.001 0.001 0.001"/>
+                <mesh filename="package://robot_one/description/meshes/gearbox.stl" scale="0.001 0.001 0.001"/>
             </geometry>
         </collision> -->
@@ -51,5 +51,5 @@
             <origin xyz="0 0 0" rpy="${pi/2} 0 ${pi}"/>
             <geometry>
-                <mesh filename="package://robot_one/meshes/gearbox.stl" scale="0.001 0.001 0.001"/>
+                <mesh filename="package://robot_one/description/meshes/gearbox.stl" scale="0.001 0.001 0.001"/>
             </geometry>
             <material name="Gazebo/blue"/>
@@ -57,5 +57,5 @@
         <!-- <collision>
             <geometry>
-               <mesh filename="package://robot_one/meshes/gearbox.stl" scale="0.001 0.001 0.001"/>
+               <mesh filename="package://robot_one/description/meshes/gearbox.stl" scale="0.001 0.001 0.001"/>
             </geometry>
         </collision> -->
@@ -73,5 +73,5 @@
         <visual>
             <geometry>
-                <mesh filename="package://robot_one/meshes/gearbox.stl" scale="0.001 0.001 0.001"/>
+                <mesh filename="package://robot_one/description/meshes/gearbox.stl" scale="0.001 0.001 0.001"/>
             </geometry>
             <material name="Gazebo/blue"/>
@@ -79,5 +79,5 @@
         <!-- <collision>
             <geometry>
-                <mesh filename="package://robot_one/meshes/gearbox.stl" scale="0.001 0.001 0.001"/>
+                <mesh filename="package://robot_one/description/meshes/gearbox.stl" scale="0.001 0.001 0.001"/>
             </geometry>
         </collision> -->

Commit message: Change publish topic name

File: description/robot_core.xacro (robot description, xacro)
@@ -30,5 +30,5 @@
                 <mesh filename="package://robot_one/description/meshes/chassis.stl" scale="0.001 0.001 0.001"/>
             </geometry>
-            <material name="Gazebo/white"/>
+            <material name="white"/>
         </visual>
         <!-- <collision>
@@ -53,5 +53,5 @@
                 <mesh filename="package://robot_one/description/meshes/gearbox.stl" scale="0.001 0.001 0.001"/>
             </geometry>
-            <material name="Gazebo/blue"/>
+            <material name="blue"/>
         </visual>
         <!-- <collision>
@@ -75,5 +75,5 @@
                 <mesh filename="package://robot_one/description/meshes/gearbox.stl" scale="0.001 0.001 0.001"/>
             </geometry>
-            <material name="Gazebo/blue"/>
+            <material name="blue"/>
         </visual>
         <!-- <collision>
